File: abra-PCB-v3/keyboard.kicad_pcb (KiCad board)
At the start: 2 copper layers, 322.3 x 131.8 mm, 166 parts

Commit message: v4 update - footprint fix
Parts:
- added U1: ATmega32U4-AU, Package_QFP:TQFP-44_10x10mm_P0.8mm, F.Cu at (290.8, 62.2)
- K_0, K_1, K_10, K_11, K_12, K_13, K_14, K_15, K_16, K_17, K_18, K_19, K_2, K_20, K_21, K_22, K_23, K_24, K_25, K_26, K_28, K_3, K_30, K_31, K_32, K_33, K_34, K_35, K_36, K_37, K_38, K_39, K_4, K_40, K_41, K_43, K_46, K_47, K_48, K_49, K_5, K_50, K_51, K_52, K_53, K_54, K_55, K_56, K_58, K_6, K_60, K_61, K_62, K_63, K_64, K_65, K_66, K_67, K_68, K_69, K_7, K_71, K_72, K_77, K_78, K_79, K_8, K_80, K_81, K_82, K_9: footprint MX_Alps_Hybrid:MX-1U-NoLED -> MX_Only:MXOnly-1U
- K_27: footprint MX_Alps_Hybrid:MX-2U-NoLED -> MX_Only:MXOnly-2U
- K_29, K_42: footprint MX_Alps_Hybrid:MX-1.5U-NoLED -> MX_Only:MXOnly-1.25U
- K_44, K_70: footprint MX_Alps_Hybrid:MX-1.75U-NoLED -> MX_Only:MXOnly-1.75U
- K_45, K_73, K_74, K_75: footprint MX_Alps_Hybrid:MX-1.25U-NoLED -> MX_Only:MXOnly-1.25U
- K_57, K_59: footprint MX_Alps_Hybrid:MX-2.25U-NoLED -> MX_Only:MXOnly-2.25U
- K_76: footprint MX_Alps_Hybrid:MX-6.25U-NoLED -> MX_Only:MXOnly-6.25U
