File: abra-PCB-v3/keyboard.sch (KiCad schematic (older format))
At the start: 250 parts

Commit message: v4 update - footprint fix
Parts:
- removed D_0, D_1, D_10, D_11, D_12, D_13, D_14, D_15, D_16, D_17, D_18, D_19, D_2, D_20, D_21, D_22, D_23, D_24, D_25, D_26, D_27, D_28, D_29, D_3, D_30, D_31, D_32, D_33, D_34, D_35, D_36, D_37, D_38, D_39, D_4, D_40, D_41, D_42, D_43, D_44, D_45, D_46, D_47, D_48, D_49, D_5, D_50, D_51, D_52, D_53, D_54, D_55, D_56, D_57, D_58, D_59, D_6, D_60, D_61, D_62, D_63, D_64, D_65, D_66, D_67, D_68, D_69, D_7, D_70, D_71, D_72, D_73, D_74, D_75, D_76, D_77, D_78, D_79, D_8, D_80, D_81, D_82, D_9: D, Diode_SMD:D_SOD-123, symbol Device:D_Small
- removed K_0, K_1, K_10, K_11, K_12, K_13, K_14, K_15, K_16, K_17, K_18, K_19, K_2, K_20, K_21, K_22, K_23, K_24, K_25, K_26, K_28, K_3, K_30, K_31, K_32, K_33, K_34, K_35, K_36, K_37, K_38, K_39, K_4, K_40, K_41, K_43, K_46, K_47, K_48, K_49, K_5, K_50, K_51, K_52, K_53, K_54, K_55, K_56, K_58, K_6, K_60, K_61, K_62, K_63, K_64, K_65, K_66, K_67, K_68, K_69, K_7, K_71, K_72, K_77, K_78, K_79, K_8, K_80, K_81, K_82, K_9: KEYSW, MX_Alps_Hybrid:MX-1U-NoLED, symbol MX_Alps_Hybrid:MX-NoLED
- removed K_27: KEYSW, MX_Alps_Hybrid:MX-2U-NoLED, symbol MX_Alps_Hybrid:MX-NoLED
- removed K_29, K_42: KEYSW, MX_Alps_Hybrid:MX-1.5U-NoLED, symbol MX_Alps_Hybrid:MX-NoLED
- removed K_44, K_70: KEYSW, MX_Alps_Hybrid:MX-1.75U-NoLED, symbol MX_Alps_Hybrid:MX-NoLED
- removed K_45, K_73, K_74, K_75: KEYSW, MX_Alps_Hybrid:MX-1.25U-NoLED, symbol MX_Alps_Hybrid:MX-NoLED
- removed K_57, K_59: KEYSW, MX_Alps_Hybrid:MX-2.25U-NoLED, symbol MX_Alps_Hybrid:MX-NoLED
- removed K_76: KEYSW, MX_Alps_Hybrid:MX-6.25U-NoLED, symbol MX_Alps_Hybrid:MX-NoLED
- added C1, C2, C3: 0.1uF, symbol Device:C_Small
- added C4, C5: C_Small, symbol Device:C_Small
- added C6: 10uF, symbol Device:C_Small
- added C7: 1uF, symbol Device:C_Small
- added C8: 4.7nF, symbol Device:C_Small
- added D1, D10, D11, D12, D13, D14, D15, D16, D17, D18, D19, D20, D21, D22, D23, D25, D26, D27, D28, D29, D3, D30, D31, D32, D33, D34, D35, D36, D37, D38, D39, D4, D40, D41, D42, D43, D44, D45, D46, D47, D48, D49, D5, D50, D51, D52, D53, D54, D55, D56, D57, D58, D59, D6, D60, D61, D62, D63, D64, D65, D66, D67, D68, D69, D7, D70, D71, D72, D73, D74, D75, D76, D77, D78, D79, D8, D80, D81, D82, D83, D9: D_Small, symbol Device:D_Small
- added J1: USB_C_Receptacle, symbol Connector:USB_C_Receptacle
- added R1, R2: R_Small, symbol Device:R_Small
- added R3: 1M, symbol Device:R_Small
- added R4, R8: 10k, symbol Device:R_Small
- added R5, R6: 5.1k, symbol Device:R_Small
- added R7: 1.5k, symbol Device:R_Small
- added SW1: SW_Push, symbol Switch:SW_Push
- added U1: ATmega32U4-AU, symbol MCU_Microchip_ATmega:ATmega32U4-AU
- added Y1: 16MHz, symbol Device:Crystal_GND24_Small
- gave numbers to parts that had none: 2
- renumbered ' to '1, , to ,1, - to -1, . to .1, / to /1, ; to ;1, = to =1, A to A1, B to B1, BCKSPACE to BCKSPACE1, C to C9, CAPS to CAPS1, D to D24, DEL to DEL1, DOWN to DOWN1, E to E1, END to END1, ENTER to ENTER1, ESC to ESC1, F to F13, FN to FN1, G to G1, H to H1, HOME to HOME1, I to I1, J to J2, K to K1, L to L1, LALT to LALT1, LCTRL to LCTRL1, LEFT to LEFT1, LSHIFT to LSHIFT1, M to M1, N to N1, O to O1, P to P1, PRTSCN to PRTSCN1, Q to Q1, R to R9, RALT to RALT1, RCTRL to RCTRL1, RIGHT to RIGHT1, RSHIFT to RSHIFT1, S to S1, SPACE to SPACE1, STPCAPS to STPCAPS1, T to T1, TAB to TAB1, U to U2, UP to UP1, V to V1, W to W1, WIN to WIN1, X to X1, Y to Y2, Z to Z1, [ to [1, \ to \1, ] to ]1, ` to `1
Connections:
- net C0: now reaches ESC1.1 (COL)
- net C0: now also CAPS1.1 (COL), LCTRL1.1 (COL), LSHIFT1.1 (COL), STPCAPS1.1 (COL), TAB1.1 (COL), `1.1 (COL)
- net C2: now reaches F1.1 (COL)
- net C2: now also LALT1.1 (COL), NUM2.1 (COL), S1.1 (COL), W1.1 (COL), X1.1 (COL)
- net at F1.2 (ROW): now also D7.2 (A)
- net C3: now reaches F2.1 (COL)
- net C3: now also C9.1 (COL), D24.1 (COL), E1.1 (COL), NUM3.1 (COL)
- net at F2.2 (ROW): now also D13.2 (A)
- net C4: now reaches F3.1 (COL)
- net C4: now also F13.1 (COL), NUM4.1 (COL), R9.1 (COL), V1.1 (COL)
- net at F3.2 (ROW): now also D19.2 (A)
- net C5: now reaches F4.1 (COL)
- net C5: now also B1.1 (COL), G1.1 (COL), NUM5.1 (COL), SPACE1.1 (COL), T1.1 (COL)
- net at F4.2 (ROW): now also D25.2 (A)
- net C6: now reaches F5.1 (COL)
- net C6: now also H1.1 (COL), N1.1 (COL), NUM6.1 (COL), Y2.1 (COL)
- net at F5.2 (ROW): now also D30.2 (A)
- net C7: now reaches F6.1 (COL)
- net C7: now also J2.1 (COL), M1.1 (COL), NUM7.1 (COL), U2.1 (COL)
- net at F6.2 (ROW): now also D36.2 (A)
- net C8: now reaches F7.1 (COL)
- net C8: now also ,1.1 (COL), I1.1 (COL), K1.1 (COL), NUM8.1 (COL)
- net at F7.2 (ROW): now also D41.2 (A)
- net C9: now reaches F8.1 (COL)
- net C9: now also .1.1 (COL), L1.1 (COL), NUM9.1 (COL), O1.1 (COL), RALT1.1 (COL)
- net at F8.2 (ROW): now also D46.2 (A)
- net C10: now reaches F9.1 (COL)
- net C10: now also /1.1 (COL), ;1.1 (COL), FN1.1 (COL), NUM0.1 (COL), P1.1 (COL)
- net at F9.2 (ROW): now also D51.2 (A)
- net C11: now reaches F10.1 (COL)
- net C11: now also '1.1 (COL), -1.1 (COL), RCTRL1.1 (COL), RSHIFT1.1 (COL), [1.1 (COL)
- net at F10.2 (ROW): now also D57.2 (A)
- net C12: now reaches F11.1 (COL)
- net C12: now also =1.1 (COL), ENTER1.1 (COL), LEFT1.1 (COL), ]1.1 (COL)
- net at F11.2 (ROW): now also D63.2 (A)
- net C13: now reaches F12.1 (COL)
- net C13: now also BCKSPACE1.1 (COL), DOWN1.1 (COL), UP1.1 (COL), \1.1 (COL)
- net at F12.2 (ROW): now also D69.2 (A)
- net ENCA: now reaches SW2.A
- net ENCB: now reaches SW2.B
- net GND: now reaches SW2.C
- net GND: now also C1.2, C2.2, C3.2, C4.2, C5.2, C6.2, C7.2, C8.2, J1.A1 (GND), J1.A12 (GND), J1.B1 (GND), J1.B12 (GND), R3.2, R5.1, R6.1, R8.1, SW1.1, U1.15 (GND), U1.23 (GND), U1.35 (GND), U1.43 (GND), U1.5 (UGND), Y1.2, Y1.4
- net C14: now reaches SW2.S1
- net C14: now also DEL1.1 (COL), END1.1 (COL), HOME1.1 (COL), PRTSCN1.1 (COL), RIGHT1.1 (COL)
- net at SW2.S2: now also D78.2 (A)
- net at `1.2 (ROW): now also D3.2 (A)
- net C1: now reaches NUM1.1 (COL)
- net C1: now also A1.1 (COL), Q1.1 (COL), WIN1.1 (COL), Z1.1 (COL)
- net at NUM1.2 (ROW): now also D8.2 (A)
- net at NUM2.2 (ROW): now also D14.2 (A)
- net at NUM3.2 (ROW): now also D20.2 (A)
- net at NUM4.2 (ROW): now also D26.2 (A)
- net at NUM5.2 (ROW): now also D31.2 (A)
- net at NUM6.2 (ROW): now also D37.2 (A)
- net at NUM7.2 (ROW): now also D42.2 (A)
- net at NUM8.2 (ROW): now also D47.2 (A)
- net at NUM9.2 (ROW): now also D52.2 (A)
- net at NUM0.2 (ROW): now also D58.2 (A)
- net at -1.2 (ROW): now also D64.2 (A)
- net at =1.2 (ROW): now also D70.2 (A)
- net at BCKSPACE1.2 (ROW): now also D74.2 (A)
- net at DEL1.2 (ROW): now also D79.2 (A)
- net at TAB1.2 (ROW): now also D4.2 (A)
- net at Q1.2 (ROW): now also D9.2 (A)
- net at W1.2 (ROW): now also D15.2 (A)
- net at E1.2 (ROW): now also D21.2 (A)
- net at R9.2 (ROW): now also D27.2 (A)
- net at T1.2 (ROW): now also D32.2 (A)
- net at Y2.2 (ROW): now also D38.2 (A)
- net at U2.2 (ROW): now also D43.2 (A)
- net at I1.2 (ROW): now also D48.2 (A)
- net at O1.2 (ROW): now also D53.2 (A)
- net at P1.2 (ROW): now also D59.2 (A)
- net at [1.2 (ROW): now also D65.2 (A)
- net at ]1.2 (ROW): now also D71.2 (A)
- net at \1.2 (ROW): now also D75.2 (A)
- net at PRTSCN1.2 (ROW): now also D80.2 (A)
- net at STPCAPS1.2 (ROW): now also CAPS1.2 (ROW), D1.2 (A)
- net at A1.2 (ROW): now also D10.2 (A)
- net at S1.2 (ROW): now also D16.2 (A)
- net at D24.2 (ROW): now also D22.2 (A)
- net at F13.2 (ROW): now also D28.2 (A)
- net at G1.2 (ROW): now also D33.2 (A)
- net at H1.2 (ROW): now also D39.2 (A)
- net at J2.2 (ROW): now also D44.2 (A)
- net at K1.2 (ROW): now also D49.2 (A)
- net at L1.2 (ROW): now also D54.2 (A)
- net at ;1.2 (ROW): now also D60.2 (A)
- net at '1.2 (ROW): now also D66.2 (A)
- net at ENTER1.2 (ROW): now also D72.2 (A)
- net at HOME1.2 (ROW): now also D81.2 (A)
- net at LSHIFT1.2 (ROW): now also D5.2 (A)
- net at Z1.2 (ROW): now also D11.2 (A)
- net at X1.2 (ROW): now also D17.2 (A)
- net at C9.2 (ROW): now also D23.2 (A)
- net at V1.2 (ROW): now also D29.2 (A)
- net at B1.2 (ROW): now also D34.2 (A)
- net at N1.2 (ROW): now also D40.2 (A)
- net at M1.2 (ROW): now also D45.2 (A)
- net at ,1.2 (ROW): now also D50.2 (A)
- net at .1.2 (ROW): now also D55.2 (A)
- net at /1.2 (ROW): now also D61.2 (A)
- net at RSHIFT1.2 (ROW): now also D67.2 (A)
- net at UP1.2 (ROW): now also D76.2 (A)
- net at END1.2 (ROW): now also D82.2 (A)
- net at LCTRL1.2 (ROW): now also D6.2 (A)
- net at WIN1.2 (ROW): now also D12.2 (A)
- net at LALT1.2 (ROW): now also D18.2 (A)
- net at SPACE1.2 (ROW): now also D35.2 (A)
- net at RALT1.2 (ROW): now also D56.2 (A)
- net at FN1.2 (ROW): now also D62.2 (A)
- net at RCTRL1.2 (ROW): now also D68.2 (A)
- net at LEFT1.2 (ROW): now also D73.2 (A)
- net at DOWN1.2 (ROW): now also D77.2 (A)
- net at RIGHT1.2 (ROW): now also D83.2 (A)
- net R0: now reaches D2.1 (K)
- net R0: now also D13.1 (K), D19.1 (K), D25.1 (K), D30.1 (K), D36.1 (K), D41.1 (K), D46.1 (K), D51.1 (K), D57.1 (K), D63.1 (K), D69.1 (K), D7.1 (K), D78.1 (K)
- new net: R4.2, SW1.2, U1.13 (~RESET)
- new net: C5.1, U1.16 (XTAL2), Y1.3
- new net: C4.1, U1.17 (XTAL1), Y1.1
- new net: R1.1, U1.3 (D-)
- new net: R8.2, U1.33 (~HWB~/PE2)
- new net: R2.1, U1.4 (D+)
- new net: C7.1, U1.6 (UCAP)
- new net: J1.A5 (CC1), R5.2
- new net: J1.A6 (D+), J1.B6 (D+), R7.2
- new net: J1.B5 (CC2), R6.2
- new net: C8.1, J1.S1 (SHIELD), R3.1
- new net +5V: C1.1, C2.1, C3.1, C6.1, R4.1, U1.14 (VCC), U1.2 (UVCC), U1.24 (AVCC), U1.34 (VCC), U1.44 (AVCC), U1.7 (VBUS)
- new net D+: R2.2, R7.1
- new net D-: J1.A7 (D-), J1.B7 (D-), R1.2
- new net R1: D14.1 (K), D20.1 (K), D26.1 (K), D3.1 (K), D31.1 (K), D37.1 (K), D42.1 (K), D47.1 (K), D52.1 (K), D58.1 (K), D64.1 (K), D70.1 (K), D74.1 (K), D79.1 (K), D8.1 (K)
- new net R2: D15.1 (K), D21.1 (K), D27.1 (K), D32.1 (K), D38.1 (K), D4.1 (K), D43.1 (K), D48.1 (K), D53.1 (K), D59.1 (K), D65.1 (K), D71.1 (K), D75.1 (K), D80.1 (K), D9.1 (K)
- new net R3: D1.1 (K), D10.1 (K), D16.1 (K), D22.1 (K), D28.1 (K), D33.1 (K), D39.1 (K), D44.1 (K), D49.1 (K), D54.1 (K), D60.1 (K), D66.1 (K), D72.1 (K), D81.1 (K)
- new net R4: D11.1 (K), D17.1 (K), D23.1 (K), D29.1 (K), D34.1 (K), D40.1 (K), D45.1 (K), D5.1 (K), D50.1 (K), D55.1 (K), D61.1 (K), D67.1 (K), D76.1 (K), D82.1 (K)
- new net R5: D12.1 (K), D18.1 (K), D35.1 (K), D56.1 (K), D6.1 (K), D62.1 (K), D68.1 (K), D73.1 (K), D77.1 (K), D83.1 (K)
- new net VBUS: J1.A4 (VBUS), J1.A9 (VBUS), J1.B4 (VBUS), J1.B9 (VBUS)
- no-connect marks 0 -> 10
Other:
- moved on the sheet: '1, ,1, -1, .1, /1, ;1, =1, A1, B1, BCKSPACE1, C9, CAPS1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
