File: abra-PCB-v4/keyboard-2.kicad_pcb (KiCad board)
At the start: 2 copper layers, 324.3 x 133 mm, 295 parts, among them J2 Conn_01x04, P1 TC2030-AVR, Q1 Q_NPN_BCE, SW1 Rotary_Encoder_Switch, SW2 SW_Push, U1 ATmega32U4-AU, U2 PRTR5V0U2X, Y1 16MHz

Commit message: routing updates
Parts:
- moved C14 6.40 mm to (154.0, 113.5)
- moved C9 6.40 mm to (142.1, 113.5)
- moved C10 6.40 mm to (144.5, 113.5)
- moved C11 6.40 mm to (146.8, 113.5)
- moved C12 6.40 mm to (149.2, 113.5)
- moved C13 6.40 mm to (151.6, 113.5)
- moved C15 6.40 mm to (156.4, 113.5)
- moved C16 6.40 mm to (158.8, 113.5)
- moved C17 6.40 mm to (161.1, 113.5)
- moved C18 6.40 mm to (163.5, 113.5)
Connections:
- K_46 pad 3: +5V -> Net-(K_46-Pad3)
- K_47 pad 3: +5V -> Net-(K_46-Pad3)
- K_48 pad 3: +5V -> Net-(K_46-Pad3)
- K_49 pad 3: +5V -> Net-(K_46-Pad3)
- K_50 pad 3: +5V -> Net-(K_46-Pad3)
- K_51 pad 3: +5V -> Net-(K_46-Pad3)
- K_52 pad 3: +5V -> Net-(K_46-Pad3)
- K_53 pad 3: +5V -> Net-(K_46-Pad3)
- K_54 pad 3: +5V -> Net-(K_46-Pad3)
- K_55 pad 3: +5V -> Net-(K_46-Pad3)
- K_56 pad 3: +5V -> Net-(K_46-Pad3)
- K_57 pad 3: +5V -> Net-(K_46-Pad3)
- K_58 pad 3: +5V -> Net-(K_46-Pad3)
- U1 pad 36: col0 -> Net-(U1-Pad36)
- U1 pad 37: col1 -> Net-(U1-Pad37)
- U1 pad 38: col2 -> Net-(U1-Pad38)
- U1 pad 39: col3 -> Net-(U1-Pad39)
- U1 pad 40: col4 -> Net-(U1-Pad40)
- U1 pad 41: col5 -> Net-(U1-Pad41)
Routing:
- net +5V: track 2093.0 -> 1579.5 mm
- net col0: track 450.1 -> 110.9 mm, vias 3 -> 0
- net col1: track 371.1 -> 93.4 mm, vias 2 -> 0
- net col2: track 366.1 -> 114.8 mm, vias 2 -> 0
- net Net-(K_46-Pad3): track 0.00 -> 233.1 mm
- net col3: track 289.3 -> 90.8 mm, vias 2 -> 0
- net col4: track 255.1 -> 90.8 mm, vias 2 -> 0
- net col6: track 246.6 -> 94.8 mm
- net col7: track 226.3 -> 94.8 mm
- net col5: track 226.4 -> 110.9 mm, vias 2 -> 0
- net col8: track 206.0 -> 94.8 mm
- net GND: track 105.1 -> 0.00 mm
- net col9: track 206.4 -> 115.8 mm
- net col11: track 177.6 -> 115.8 mm
- net col10: track 180.3 -> 119.7 mm
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