File: abra-PCB-v4/keyboard.kicad_pcb (KiCad board)
At the start: 2 copper layers, 166 parts, among them SW1 Rotary_Encoder_Switch

Commit message: layout changes
Parts:
- removed D_44: D, Diode_SMD:D_SOD-123
- added C1: 0.1uF, acheron_Components:C_0805_2012Metric, B.Cu at (410.2, 158.8)
- added C10: 0.1uF, acheron_Components:C_0805_2012Metric, B.Cu at (358.8, 17.5)
- added C11: 0.1uF, acheron_Components:C_0805_2012Metric, B.Cu at (358.8, 12.7)
- added C12: 0.1uF, acheron_Components:C_0805_2012Metric, B.Cu at (358.8, 7.14)
- added C13: 0.1uF, acheron_Components:C_0805_2012Metric, B.Cu at (358.8, 1.59)
- added C14: 0.1uF, acheron_Components:C_0805_2012Metric, B.Cu at (358.8, -3.97)
- added C15: 0.1uF, acheron_Components:C_0805_2012Metric, B.Cu at (358.8, -9.53)
- added C16: 0.1uF, acheron_Components:C_0805_2012Metric, B.Cu at (144.5, -148.4)
- added C17: 0.1uF, acheron_Components:C_0805_2012Metric, B.Cu at (232.3, 18.7)
- added C18: 0.1uF, acheron_Components:C_0805_2012Metric, B.Cu at (227.9, 18.7)
- added C19: 0.1uF, acheron_Components:C_0805_2012Metric, B.Cu at (218.0, 8.75)
- added C2: 22pF, acheron_Components:C_0805_2012Metric, B.Cu at (421.5, 158.0)
- added C20: 0.1uF, acheron_Components:C_0805_2012Metric, B.Cu at (251.4, 41.7)
- added C3: 22pF, acheron_Components:C_0805_2012Metric, B.Cu at (420.7, 154.0)
- added C4: 1uF, acheron_Components:C_0805_2012Metric, B.Cu at (238.7, 28.6)
- added C5: 0.1uF, acheron_Components:C_0805_2012Metric, B.Cu at (410.2, 161.1)
- added C6: 0.1uF, acheron_Components:C_0805_2012Metric, B.Cu at (410.2, 156.4)
- added C7: 10uF, acheron_Components:C_0805_2012Metric, B.Cu at (410.2, 154.0)
- added C8: 4.7uF, acheron_Components:C_0805_2012Metric, B.Cu at (222.4, 8.75)
- added C9: 0.1uF, acheron_Components:C_0805_2012Metric, B.Cu at (358.8, 21.4)
- added D1: WS2812B, LED_SMD:LED_WS2812B_PLCC4_5.0x5.0mm_P3.2mm, B.Cu at (130.2, 130.2)
- added D10: WS2812B, LED_SMD:LED_WS2812B_PLCC4_5.0x5.0mm_P3.2mm, B.Cu at (437.4, 171.4)
- added D11: WS2812B, LED_SMD:LED_WS2812B_PLCC4_5.0x5.0mm_P3.2mm, B.Cu at (437.4, 190.5)
- added D12: WS2812B, LED_SMD:LED_WS2812B_PLCC4_5.0x5.0mm_P3.2mm, B.Cu at (437.4, 198.4)
- added D2: WS2812B, LED_SMD:LED_WS2812B_PLCC4_5.0x5.0mm_P3.2mm, B.Cu at (130.2, 140.5)
- added D3: WS2812B, LED_SMD:LED_WS2812B_PLCC4_5.0x5.0mm_P3.2mm, B.Cu at (130.2, 150.8)
- added D4: WS2812B, LED_SMD:LED_WS2812B_PLCC4_5.0x5.0mm_P3.2mm, B.Cu at (130.2, 161.1)
- added D5: WS2812B, LED_SMD:LED_WS2812B_PLCC4_5.0x5.0mm_P3.2mm, B.Cu at (130.2, 171.4)
- added D6: WS2812B, LED_SMD:LED_WS2812B_PLCC4_5.0x5.0mm_P3.2mm, B.Cu at (130.2, 181.0)
- added D7: WS2812B, LED_SMD:LED_WS2812B_PLCC4_5.0x5.0mm_P3.2mm, B.Cu at (437.4, 113.5)
- added D8: WS2812B, LED_SMD:LED_WS2812B_PLCC4_5.0x5.0mm_P3.2mm, B.Cu at (437.4, 133.3)
- added D9: WS2812B, LED_SMD:LED_WS2812B_PLCC4_5.0x5.0mm_P3.2mm, B.Cu at (437.4, 152.4)
- added F1: 500mA Hold, acheron_Components:Fuse_1812_4532, B.Cu at (189.6, 23.8)
- added J2: Conn_01x04, Connector_PinHeader_2.54mm:PinHeader_1x04_P2.54mm_Vertical_SMD_Pin1Left, B.Cu at (146.5, 60.9)
- added P1: TC2030-AVR, Keebio-Parts:Header-6-Pin-ZigZag, B.Cu at (174.0, 50.8)
- added Q1: Q_NPN_BCE, Package_TO_SOT_SMD:SOT-223-3_TabPin2, B.Cu at (176.6, 17.2)
- added R1: 22, acheron_Components:R_SMD_1206, B.Cu at (222.4, 41.6)
- added R10: R_Small, acheron_Components:R_SMD_1206, B.Cu at (214.4, 34.9)
- added R11: R_Small, acheron_Components:R_SMD_1206, B.Cu at (220.3, 35.0)
- added R12: R_Small, acheron_Components:R_SMD_1206, B.Cu at (226.3, 38.3)
- added R13: R_Small, acheron_Components:R_SMD_1206, B.Cu at (215.7, 28.3)
- added R14: R_Small, acheron_Components:R_SMD_1206, B.Cu at (222.4, 48.1)
- added R15: R_Small, acheron_Components:R_SMD_1206, B.Cu at (204.9, 18.4)
- added R16: R_Small, acheron_Components:R_SMD_1206, B.Cu at (228.3, 41.6)
- added R17: R_Small, acheron_Components:R_SMD_1206, B.Cu at (201.0, 13.4)
- added R18: R_Small, acheron_Components:R_SMD_1206, B.Cu at (234.3, 44.9)
- added R19: R_Small, acheron_Components:R_SMD_1206, B.Cu at (210.8, 21.7)
- added R2: 22, acheron_Components:R_SMD_1206, B.Cu at (195.0, 13.1)
- added R20: R_Small, acheron_Components:R_SMD_1206, B.Cu at (240.2, 51.4)
- added R21: R_Small, acheron_Components:R_SMD_1206, B.Cu at (215.7, 25.0)
- added R22: R_Small, acheron_Components:R_SMD_1206, B.Cu at (203.8, 28.3)
- added R23: R_Small, acheron_Components:R_SMD_1206, B.Cu at (216.4, 51.4)
- added R24: R_Small, acheron_Components:R_SMD_1206, B.Cu at (216.4, 48.1)
- added R25: R_Small, acheron_Components:R_SMD_1206, B.Cu at (183.1, 11.4)
- added R26: R_Small, acheron_Components:R_SMD_1206, B.Cu at (216.4, 44.9)
- added R27: R_Small, acheron_Components:R_SMD_1206, B.Cu at (222.4, 51.4)
- added R28: R_Small, acheron_Components:R_SMD_1206, B.Cu at (193.0, 19.7)
- added R29: R_Small, acheron_Components:R_SMD_1206, B.Cu at (203.8, 31.6)
- added R3: 10k, acheron_Components:R_SMD_1206, B.Cu at (228.3, 44.9)
- added R30: R_Small, acheron_Components:R_SMD_1206, B.Cu at (224.8, 15.2)
- added R31: R_Small, acheron_Components:R_SMD_1206, B.Cu at (227.6, 31.7)
- added R32: R_Small, acheron_Components:R_SMD_1206, B.Cu at (221.7, 31.7)
- added R33: R_Small, acheron_Components:R_SMD_1206, B.Cu at (212.9, 15.1)
- added R34: R_Small, acheron_Components:R_SMD_1206, B.Cu at (232.2, 35.0)
- added R35: R_Small, acheron_Components:R_SMD_1206, B.Cu at (238.2, 38.3)
- added R36: R_Small, acheron_Components:R_SMD_1206, B.Cu at (227.6, 28.4)
- added R37: R_Small, acheron_Components:R_SMD_1206, B.Cu at (216.8, 18.5)
- added R38: R_Small, acheron_Components:R_SMD_1206, B.Cu at (206.9, 8.54)
- added R39: R_Small, acheron_Components:R_SMD_1206, B.Cu at (240.2, 41.6)
- added R4: 1M, acheron_Components:R_SMD_1206, B.Cu at (198.9, 16.7)
- added R40: R_Small, acheron_Components:R_SMD_1206, B.Cu at (246.2, 44.9)
- added R41: R_Small, acheron_Components:R_SMD_1206, B.Cu at (212.9, 11.8)
- added R42: R_Small, acheron_Components:R_SMD_1206, B.Cu at (222.7, 21.8)
- added R43: R_Small, acheron_Components:R_SMD_1206, B.Cu at (252.1, 51.4)
- added R44: R_Small, acheron_Components:R_SMD_1206, B.Cu at (227.6, 25.1)
- added R45: R_Small, acheron_Components:R_SMD_1206, B.Cu at (233.6, 31.7)
- added R46: R_Small, acheron_Components:R_SMD_1206, B.Cu at (222.4, 44.9)
- added R47: R_Small, acheron_Components:R_SMD_1206, B.Cu at (220.3, 38.3)
- added R48: R_Small, acheron_Components:R_SMD_1206, B.Cu at (209.8, 28.3)
- added R49: R_Small, acheron_Components:R_SMD_1206, B.Cu at (196.1, 23.3)
- added R5: 10k, acheron_Components:R_SMD_1206, B.Cu at (234.3, 51.4)
- added R50: R_Small, acheron_Components:R_SMD_1206, B.Cu at (214.4, 38.2)
- added R51: R_Small, acheron_Components:R_SMD_1206, B.Cu at (179.3, 37.9)
- added R52: R_Small, acheron_Components:R_SMD_1206, B.Cu at (216.4, 41.6)
- added R53: R_Small, acheron_Components:R_SMD_1206, B.Cu at (183.1, 8.09)
- added R54: R_Small, acheron_Components:R_SMD_1206, B.Cu at (189.1, 13.0)
- added R55: R_Small, acheron_Components:R_SMD_1206, B.Cu at (228.3, 48.1)
- added R56: R_Small, acheron_Components:R_SMD_1206, B.Cu at (195.0, 9.81)
- added R57: R_Small, acheron_Components:R_SMD_1206, B.Cu at (228.3, 51.4)
- added R58: R_Small, acheron_Components:R_SMD_1206, B.Cu at (198.9, 20.0)
- added R59: R_Small, acheron_Components:R_SMD_1206, B.Cu at (203.8, 25.0)
- added R6: 5.1k, acheron_Components:R_SMD_1206, B.Cu at (204.9, 21.7)
- added R60: R_Small, acheron_Components:R_SMD_1206, B.Cu at (209.8, 31.6)
- added R61: R_Small, acheron_Components:R_SMD_1206, B.Cu at (216.8, 21.7)
- added R62: R_Small, acheron_Components:R_SMD_1206, B.Cu at (193.0, 16.4)
- added R63: R_Small, acheron_Components:R_SMD_1206, B.Cu at (252.1, 48.1)
- added R64: R_Small, acheron_Components:R_SMD_1206, B.Cu at (189.1, 9.72)
- added R65: R_Small, acheron_Components:R_SMD_1206, B.Cu at (218.8, 15.2)
- added R66: R_Small, acheron_Components:R_SMD_1206, B.Cu at (246.2, 48.1)
- added R67: R_Small, acheron_Components:R_SMD_1206, B.Cu at (244.1, 38.3)
- added R68: R_Small, acheron_Components:R_SMD_1206, B.Cu at (233.6, 28.4)
- added R69: R_Small, acheron_Components:R_SMD_1206, B.Cu at (222.7, 18.5)
- added R7: 5.1k, acheron_Components:R_SMD_1206, B.Cu at (209.8, 25.0)
- added R70: R_Small, acheron_Components:R_SMD_1206, B.Cu at (212.9, 8.54)
- added R71: R_Small, acheron_Components:R_SMD_1206, B.Cu at (246.2, 41.6)
- added R72: R_Small, acheron_Components:R_SMD_1206, B.Cu at (252.1, 44.9)
- added R73: R_Small, acheron_Components:R_SMD_1206, B.Cu at (218.8, 11.9)
- added R74: R_Small, acheron_Components:R_SMD_1206, B.Cu at (228.7, 21.8)
- added R75: R_Small, acheron_Components:R_SMD_1206, B.Cu at (233.6, 25.1)
- added R76: R_Small, acheron_Components:R_SMD_1206, B.Cu at (239.5, 31.7)
- added R77: R_Small, acheron_Components:R_SMD_1206, B.Cu at (244.1, 35.0)
- added R78: R_Small, acheron_Components:R_SMD_1206, B.Cu at (238.2, 35.0)
- added R79: R_Small, acheron_Components:R_SMD_1206, B.Cu at (221.7, 25.1)
- added R8: 500, acheron_Components:R_SMD_1206, B.Cu at (215.7, 31.6)
- added R80: R_Small, acheron_Components:R_SMD_1206, B.Cu at (240.2, 48.1)
- added R81: R_Small, acheron_Components:R_SMD_1206, B.Cu at (201.0, 10.2)
- added R82: R_Small, acheron_Components:R_SMD_1206, B.Cu at (226.3, 35.0)
- added R83: R_Small, acheron_Components:R_SMD_1206, B.Cu at (232.2, 38.3)
- added R84: R_Small, acheron_Components:R_SMD_1206, B.Cu at (221.7, 28.4)
- added R85: R_Small, acheron_Components:R_SMD_1206, B.Cu at (210.8, 18.4)
- added R86: R_Small, acheron_Components:R_SMD_1206, B.Cu at (234.3, 41.6)
- added R87: R_Small, acheron_Components:R_SMD_1206, B.Cu at (206.9, 15.1)
- added R88: R_Small, acheron_Components:R_SMD_1206, B.Cu at (240.2, 44.9)
- added R89: R_Small, acheron_Components:R_SMD_1206, B.Cu at (206.9, 11.8)
- added R9: 1.5k, acheron_Components:R_SMD_1206, B.Cu at (234.3, 48.1)
- added R90: R_Small, acheron_Components:R_SMD_1206, B.Cu at (246.2, 51.4)
- added R91: 22, acheron_Components:R_SMD_1206, B.Cu at (153.4, 55.7)
- added R92: 22, acheron_Components:R_SMD_1206, B.Cu at (164.5, 65.4)
- added SW2: SW_Push, random-keyboard-parts:Reset_Pretty, B.Cu at (197.7, 29.3)
- added U1: ATmega32U4-AU, Package_QFP:TQFP-44_10x10mm_P0.8mm, B.Cu at (418.3, 171.4)
- added U2: PRTR5V0U2X, Nexperia:SOT143B, B.Cu at (249.1, 30.5)
- added USB1: HRO-TYPE-C-31-M-12, Type-C:HRO-TYPE-C-31-M-12-HandSoldering, B.Cu at (417.5, 99.2)
- added Y1: 16MHz, Keebio-Parts:Crystal_SMD_3225-4pin_3.2x2.5mm, B.Cu at (417.5, 158.0)
- K_0, K_1, K_10, K_11, K_12, K_14, K_15, K_16, K_17, K_18, K_19, K_2, K_20, K_21, K_22, K_23, K_24, K_25, K_26, K_28, K_3, K_30, K_31, K_32, K_33, K_34, K_35, K_36, K_37, K_38, K_39, K_4, K_40, K_41, K_43, K_46, K_47, K_48, K_49, K_5, K_50, K_51, K_52, K_53, K_54, K_55, K_56, K_58, K_6, K_60, K_61, K_62, K_63, K_64, K_65, K_66, K_67, K_68, K_69, K_7, K_71, K_72, K_77, K_78, K_79, K_8, K_80, K_81, K_82, K_9: footprint MX_Only:MXOnly-1U-NoLED -> MX_Only:MXOnly-1U
- K_27: footprint MX_Only:MXOnly-2U-NoLED -> MX_Only:MXOnly-2U
- K_29, K_42: footprint MX_Only:MXOnly-1.5U-NoLED -> MX_Only:MXOnly-1.5U
- K_44, K_70: footprint MX_Only:MXOnly-1.75U-NoLED -> MX_Only:MXOnly-1.75U
- K_45: value KEYSW -> MX-NoLED; footprint MX_Only:MXOnly-1.25U-NoLED -> MX_Only:MXOnly-1.75U-NoLED
- K_57, K_59: footprint MX_Only:MXOnly-2.25U-NoLED -> MX_Only:MXOnly-2.25U
- K_73, K_74, K_75: footprint MX_Only:MXOnly-1.25U-NoLED -> MX_Only:MXOnly-1.25U
- K_76: footprint MX_Only:MXOnly-6.25U-NoLED -> MX_Only:MXOnly-6.25U
- moved D_76 49.8 mm to (266.7, 201.3)
- moved D_57 11.7 mm to (400.1, 163.2)
- moved D_27 9.32 mm to (402.4, 125.1)
- moved D_42 4.56 mm to (407.2, 144.2)

Commit message: layout updates
Parts:
- K_45: footprint MX_Only:MXOnly-1.75U-NoLED -> MX_Only:MXOnly-1.75U
- moved Q1 304.9 mm to (424.7, 194.5)
- moved R89 286.1 mm to (431.0, 189.7), turned to 180 degrees
- moved R85 280.3 mm to (414.3, 211.1), turned to 270 degrees
- moved R91 273.6 mm to (422.3, 106.4), turned to 90 degrees
- moved J2 269.6 mm to (411.2, 111.9), turned to 270 degrees
- moved R92 263.3 mm to (424.7, 106.5), turned to 90 degrees
- moved C16 262.3 mm to (158.8, 113.5), turned to 270 degrees
- moved R87 259.4 mm to (427.0, 152.4), turned to 180 degrees
- moved P1 257.4 mm to (388.1, 193.7), turned to 270 degrees
- moved F1 254.2 mm to (427.8, 112.7)
- moved R84 252.0 mm to (412.0, 193.7), turned to 270 degrees
- moved R2 249.2 mm to (418.3, 123.8), turned to 90 degrees
- moved R90 246.1 mm to (433.4, 211.1), turned to 270 degrees
- moved R4 240.7 mm to (420.7, 110.3)
- moved C15 236.9 mm to (156.4, 113.5), turned to 270 degrees
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Connections:
- R21 pad 1: Net-(R21-Pad1) -> Net-(K_45-Pad4)
Other:
- board outline added: 324.3 x 133 mm

Commit message: light fix + library update
Parts:
- removed C19, C20: 0.1uF, acheron_Components:C_0805_2012Metric
- removed D11, D12: WS2812B, LED_SMD:LED_WS2812B_PLCC4_5.0x5.0mm_P3.2mm
- added R93: R_Small, acheron_Components:R_SMD_1206, B.Cu at (130.6, 113.0)
- D1, D10, D2, D3, D4, D5, D6, D7, D8, D9: value WS2812B -> SK6805; footprint LED_SMD:LED_WS2812B_PLCC4_5.0x5.0mm_P3.2mm -> LED_SMD:LED_SK6812_EC15_1.5x1.5mm
- moved D6 312.2 mm to (438.6, 132.8), turned to 0 degrees
- moved R8 39.6 mm to (163.8, 98.0)
- moved D7 28.1 mm to (438.5, 142.3), turned to 0 degrees
- moved D8 21.7 mm to (438.5, 151.9), turned to 0 degrees
- moved D9 12.1 mm to (438.5, 161.3), turned to 0 degrees
- moved D1 8.33 mm to (129.6, 138.5), turned to 0 degrees
- moved D2 7.41 mm to (129.6, 147.9), turned to 0 degrees
- moved D3 6.75 mm to (129.6, 157.5), turned to 0 degrees
- moved D4 5.78 mm to (129.6, 166.9), turned to 0 degrees
- moved D5 5.17 mm to (129.6, 176.6), turned to 0 degrees
- moved D10 3.01 mm to (438.5, 171.1), turned to 0 degrees
Connections:
- D1 pad 1: +5V -> Net-(D1-Pad1)
- D1 pad 2: Net-(D1-Pad2) -> GND
- D1 pad 3: GND -> Net-(D1-Pad3)
- D1 pad 4: Net-(D1-Pad4) -> +5V
- D10 pad 1: +5V -> Net-(D10-Pad1)
- D10 pad 2: Net-(D10-Pad2) -> GND
- D10 pad 3: GND -> Net-(D10-Pad3)
- D10 pad 4: Net-(D10-Pad4) -> +5V
- D2 pad 1: +5V -> Net-(D2-Pad1)
- D2 pad 2: Net-(D2-Pad2) -> GND
- D2 pad 3: Net-(D2-Pad3) -> Net-(D1-Pad1)
- D2 pad 4: Net-(D1-Pad2) -> +5V
- D3 pad 1: +5V -> Net-(D3-Pad1)
- D3 pad 2: Net-(D3-Pad2) -> GND
- D3 pad 3: Net-(D3-Pad3) -> Net-(D2-Pad1)
- D3 pad 4: Net-(D2-Pad2) -> +5V
- D4 pad 1: +5V -> Net-(D4-Pad1)
- D4 pad 2: Net-(D4-Pad2) -> GND
- D4 pad 3: Net-(D4-Pad3) -> Net-(D3-Pad1)
- D4 pad 4: Net-(D3-Pad2) -> +5V
- D5 pad 1: +5V -> Net-(D5-Pad1)
- D5 pad 2: Net-(D5-Pad2) -> GND
- D5 pad 3: Net-(D5-Pad3) -> Net-(D4-Pad1)
- D5 pad 4: Net-(D4-Pad2) -> +5V
- D6 pad 1: +5V -> Net-(D6-Pad1)
- D6 pad 2: Net-(D6-Pad2) -> GND
- D6 pad 3: Net-(D6-Pad3) -> Net-(D5-Pad1)
- D6 pad 4: Net-(D5-Pad2) -> +5V
- D7 pad 1: +5V -> Net-(D7-Pad1)
- D7 pad 2: Net-(D7-Pad2) -> GND
- D7 pad 3: GND -> Net-(D6-Pad1)
- D7 pad 4: Net-(D6-Pad2) -> +5V
- D8 pad 1: +5V -> Net-(D8-Pad1)
- D8 pad 2: Net-(D8-Pad2) -> GND
- D8 pad 3: Net-(D8-Pad3) -> Net-(D7-Pad1)
- D8 pad 4: Net-(D7-Pad2) -> +5V
- D9 pad 1: +5V -> Net-(D10-Pad3)
- D9 pad 2: Net-(D10-Pad4) -> GND
- D9 pad 3: GND -> Net-(D8-Pad1)
- D9 pad 4: Net-(D8-Pad2) -> +5V
- R8 pad 1: Net-(D1-Pad4) -> Net-(D1-Pad3)

Commit message: routing updates
Parts:
- moved R93 84.9 mm to (195.4, 167.9)
- moved R8 47.5 mm to (129.0, 130.3), turned to 90 degrees
- moved SW2 44.3 mm to (415.3, 138.7)
- moved R3 41.6 mm to (415.5, 149.4)
- moved D_59 12.1 mm to (156.7, 182.2)
- moved R86 9.36 mm to (436.1, 131.1), turned to 270 degrees
- moved R87 9.36 mm to (436.1, 150.1), turned to 270 degrees
- moved R88 7.83 mm to (436.1, 169.2), turned to 270 degrees
- moved R81 7.52 mm to (409.4, 105.9), turned to 0 degrees
- moved D_70 7.13 mm to (385.6, 182.3)
- moved C14 6.40 mm to (147.6, 112.7)
- moved C9 6.40 mm to (135.7, 112.7)
- moved C10 6.40 mm to (138.1, 112.7)
- moved C11 6.40 mm to (140.5, 112.7)
- moved C12 6.40 mm to (142.9, 112.7)
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Connections:
- K_46 pad 3: Net-(K_46-Pad3) -> +5V
- K_47 pad 3: Net-(K_46-Pad3) -> +5V
- K_48 pad 3: Net-(K_46-Pad3) -> +5V
- K_49 pad 3: Net-(K_46-Pad3) -> +5V
- K_50 pad 3: Net-(K_46-Pad3) -> +5V
- K_51 pad 3: Net-(K_46-Pad3) -> +5V
- K_52 pad 3: Net-(K_46-Pad3) -> +5V
- K_53 pad 3: Net-(K_46-Pad3) -> +5V
- K_54 pad 3: Net-(K_46-Pad3) -> +5V
- K_55 pad 3: Net-(K_46-Pad3) -> +5V
- K_56 pad 3: Net-(K_46-Pad3) -> +5V
- K_57 pad 3: Net-(K_46-Pad3) -> +5V
- K_58 pad 3: Net-(K_46-Pad3) -> +5V
- U1 pad 36: Net-(U1-Pad36) -> col0
- U1 pad 37: Net-(U1-Pad37) -> col1
- U1 pad 38: Net-(U1-Pad38) -> col2
- U1 pad 39: Net-(U1-Pad39) -> col3
- U1 pad 40: Net-(U1-Pad40) -> col4
- U1 pad 41: Net-(U1-Pad41) -> col5
Routing:
- net +5V: track 0.00 -> 2093.0 mm
- net col0: track 0.00 -> 450.1 mm, vias 0 -> 3
- net col1: track 0.00 -> 371.1 mm, vias 0 -> 2
- net col2: track 0.00 -> 366.1 mm, vias 0 -> 2
- net Net-(K_41-Pad4): track 0.00 -> 310.0 mm
- net Net-(R15-Pad2): track 0.00 -> 299.3 mm
- net Net-(K_80-Pad4): track 0.00 -> 299.2 mm
- net col3: track 0.00 -> 289.3 mm, vias 0 -> 2
- net row5: track 0.00 -> 289.0 mm
- net LEDGND: track 0.00 -> 282.6 mm
- net row1: track 0.00 -> 280.6 mm
- net row2: track 0.00 -> 276.1 mm
- net Net-(K_57-Pad4): track 0.00 -> 274.3 mm
- net Net-(K_70-Pad4): track 0.00 -> 273.3 mm
- net row4: track 0.00 -> 273.0 mm
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Other:
- net class Power added: clearance 0.2, trace_width 0.381, via_dia 0.8, via_drill 0.4

Commit message: routing updates
Connections:
- U1 pad 32: Net-(U1-Pad32) -> ENB1
- U1 pad 8: Net-(U1-Pad8) -> col13
Routing:
- net ENB1: track 97.3 -> 171.4 mm, vias 0 -> 2
- net col13: track 125.9 -> 191.0 mm, vias 0 -> 2
- net col2: track 366.1 -> 401.5 mm, vias 2 -> 3
- net col1: track 371.1 -> 406.3 mm, vias 2 -> 3
- net col12: track 180.0 -> 180.6 mm, vias 0 -> 1
- net col11: track 177.6 -> 178.0 mm, vias 0 -> 1

Commit message: routing updates
Connections:
- U1 pad 10: Net-(U1-Pad10) -> col11
- U1 pad 11: Net-(U1-Pad11) -> col10
- U1 pad 12: Net-(U1-Pad12) -> col9
- U1 pad 18: Net-(U1-Pad18) -> col6
- U1 pad 19: Net-(U1-Pad19) -> col7
- U1 pad 20: Net-(U1-Pad20) -> col8
- U1 pad 9: Net-(U1-Pad9) -> col12
Routing:
- net col8: track 206.0 -> 297.5 mm, vias 0 -> 2
- net col7: track 226.3 -> 315.6 mm, vias 0 -> 2
- net col6: track 246.6 -> 334.0 mm, vias 0 -> 2
- net col10: track 180.3 -> 263.2 mm, vias 0 -> 2
- net col9: track 206.4 -> 288.4 mm, vias 0 -> 2
- net col3: track 289.3 -> 362.8 mm, vias 2 -> 3
- net col11: track 178.0 -> 241.3 mm, vias 1 -> 2
- net col12: track 180.6 -> 242.9 mm, vias 1 -> 2
- net col4: track 255.1 -> 270.6 mm
- net Net-(C3-Pad1): track 0.00 -> 10.5 mm
- net Net-(C2-Pad1): track 0.00 -> 7.07 mm
- net GND: track 108.3 -> 114.1 mm

Commit message: routing updates
Parts:
- removed P1: TC2030-AVR, Keebio-Parts:Header-6-Pin-ZigZag
- SW2: footprint random-keyboard-parts:Reset_Pretty -> Keebio-Parts:SW_SPST_3x3
- moved USB1 8.92 mm to (417.6, 90.3), turned to 0 degrees
- moved R3 4.93 mm to (410.9, 151.1), turned to 0 degrees
- moved U2 3.63 mm to (421.5, 153.6), turned to 90 degrees
- moved C3 3.20 mm to (417.5, 154.2)
- moved SW2 1.67 mm to (415.0, 137.0), turned to 270 degrees
Connections:
- net RST renamed Net-(R3-Pad2)
- SW1 pad A: Net-(SW1-PadA) -> ENA
- SW1 pad B: Net-(SW1-PadB) -> ENB
- SW1 pad C: Net-(SW1-PadC) -> GND
- U1 pad 21: Net-(U1-Pad21) -> row0
- U1 pad 22: Net-(U1-Pad22) -> row1
- U1 pad 25: Net-(U1-Pad25) -> row3
- U1 pad 28: Net-(U1-Pad28) -> ENA
- U1 pad 29: Net-(U1-Pad29) -> ENB
- U1 pad 30: Net-(U1-Pad30) -> row5
- U1 pad 31: Net-(U1-Pad31) -> row4
Routing:
- net GND: track 114.1 -> 440.4 mm
- net ENB: track 0.00 -> 105.6 mm, vias 0 -> 1
- net ENA: track 0.00 -> 94.9 mm, vias 0 -> 1
- net row0: track 268.4 -> 347.3 mm, vias 0 -> 2
- net col5: track 226.4 -> 296.4 mm, vias 2 -> 3
- net row1: track 280.6 -> 340.4 mm, vias 0 -> 2
- net row5: track 289.0 -> 343.5 mm, vias 0 -> 2
- net Net-(J2-Pad2): track 0.00 -> 50.2 mm, vias 0 -> 4
- net Net-(C8-Pad1): track 0.00 -> 45.9 mm, vias 0 -> 3
- net VCC: track 0.00 -> 41.2 mm, vias 0 -> 3
- net col4: track 270.6 -> 308.3 mm, vias 2 -> 3
- net Net-(J2-Pad3): track 0.00 -> 32.6 mm, vias 0 -> 4
- net row4: track 273.0 -> 301.5 mm
- net D-: track 0.00 -> 27.7 mm
- net D+: track 0.00 -> 21.2 mm
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