File: abra-PCB-v4/keyboard-4.kicad_pcb (KiCad board)
At the start: 2 copper layers, 324.3 x 133 mm, 294 parts, among them J2 Conn_01x04, Q1 Q_NPN_BCE, SW1 Rotary_Encoder_Switch, SW2 SW_Push, U1 ATmega32U4-AU, U2 PRTR5V0U2X, Y1 16MHz

Commit message: version 4
Parts:
- moved U2 41.5 mm to (403.6, 112.4)
- moved Q1 34.4 mm to (392.9, 176.0), turned to 270 degrees
- moved R9 24.7 mm to (399.2, 174.6), turned to 270 degrees
- moved C1 13.8 mm to (396.0, 195.9)
- moved C5 13.8 mm to (398.4, 195.9)
- moved C6 13.8 mm to (393.6, 195.9)
- moved C7 13.8 mm to (391.2, 195.9)
- moved R5 4.40 mm to (416.1, 180.8)
- moved R7 2.41 mm to (413.8, 112.5)
- moved R6 2.38 mm to (411.4, 112.5)
- moved C2 1.82 mm to (424.7, 157.2)
- moved C3 1.82 mm to (419.6, 157.5)
- moved Y1 1.82 mm to (422.0, 160.0)
Connections:
- U1 pad 10: Net-(U1-Pad10) -> row2
- U1 pad 11: Net-(U1-Pad11) -> row1
- U1 pad 12: Net-(U1-Pad12) -> row0
- U1 pad 9: Net-(U1-Pad9) -> row3
Routing:
- net +5V: track 0.00 -> 1917.3 mm, vias 0 -> 3
- net Net-(K_70-Pad4): track 0.00 -> 402.4 mm, vias 0 -> 4
- net Net-(K_41-Pad4): track 0.00 -> 316.2 mm
- net Net-(K_57-Pad4): track 0.00 -> 310.9 mm
- net Net-(K_80-Pad4): track 0.00 -> 305.6 mm
- net row3: track 0.00 -> 301.5 mm, vias 0 -> 2
- net Net-(R15-Pad2): track 0.00 -> 299.2 mm
- net row0: track 0.00 -> 292.8 mm, vias 0 -> 2
- net LEDGND: track 0.00 -> 290.1 mm
- net row1: track 0.00 -> 289.9 mm, vias 0 -> 1
- net row5: track 0.00 -> 289.0 mm
- net row2: track 0.00 -> 287.1 mm, vias 0 -> 1
- net row4: track 0.00 -> 284.3 mm
- net GND: track 0.00 -> 265.1 mm, vias 0 -> 6
- net col12: track 0.00 -> 138.0 mm
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
Commit message: v4 routing complete
Parts:
- moved C14 3.39 mm to (150.9, 112.0)
- moved C9 3.39 mm to (139.0, 112.0)
- moved C10 3.39 mm to (141.4, 112.0)
- moved C11 3.39 mm to (143.8, 112.0)
- moved C12 3.39 mm to (146.2, 112.0)
- moved C13 3.39 mm to (148.6, 112.0)
- moved C15 3.39 mm to (153.3, 112.0)
- moved C16 3.39 mm to (155.7, 112.0)
- moved C17 3.39 mm to (158.1, 112.0)
- moved C18 3.39 mm to (160.5, 112.0)
Connections:
- net ENB2 renamed Net-(D_13-Pad2)
- K_28 pad 1: ENB1 -> col14
- K_43 pad 1: ENB1 -> col14
- K_58 pad 1: ENB1 -> col14
- K_71 pad 1: ENB1 -> col14
- K_82 pad 1: ENB1 -> col14
- SW1 pad S1: ENB1 -> col14
- U1 pad 11: row1 -> row3
- U1 pad 12: row0 -> row4
- U1 pad 18: Net-(U1-Pad18) -> row5
- U1 pad 19: Net-(U1-Pad19) -> ENA
- U1 pad 20: Net-(U1-Pad20) -> ENB
- U1 pad 21: Net-(U1-Pad21) -> col14
- U1 pad 22: Net-(U1-Pad22) -> col13
- U1 pad 25: Net-(U1-Pad25) -> col12
- U1 pad 26: Net-(U1-Pad26) -> col11
- U1 pad 27: Net-(U1-Pad27) -> col10
- U1 pad 28: Net-(U1-Pad28) -> col9
- U1 pad 29: Net-(U1-Pad29) -> col8
- U1 pad 30: Net-(U1-Pad30) -> col7
- U1 pad 31: Net-(U1-Pad31) -> col6
- U1 pad 32: Net-(U1-Pad32) -> col5
- U1 pad 36: Net-(U1-Pad36) -> col4
- U1 pad 37: Net-(U1-Pad37) -> col3
- U1 pad 38: Net-(U1-Pad38) -> col2
- U1 pad 39: Net-(U1-Pad39) -> col1
- U1 pad 40: Net-(U1-Pad40) -> col0
- U1 pad 41: Net-(U1-Pad41) -> RGBIN
- U1 pad 8: Net-(U1-Pad8) -> row0
- U1 pad 9: row3 -> row1
Routing:
- net +5V: track 1917.3 -> 3660.3 mm, vias 3 -> 8
- net Net-(D5-Pad1): track 0.00 -> 448.0 mm, vias 0 -> 2
- net GND: track 265.1 -> 642.4 mm
- net RGBIN: track 0.00 -> 360.9 mm, vias 0 -> 2
- net col0: track 115.6 -> 401.9 mm, vias 0 -> 3
- net col1: track 93.9 -> 349.6 mm, vias 0 -> 2
- net col2: track 114.8 -> 346.6 mm, vias 0 -> 2
- net col4: track 90.8 -> 319.9 mm, vias 0 -> 3
- net col3: track 90.8 -> 305.1 mm, vias 0 -> 2
- net col5: track 110.9 -> 306.1 mm, vias 0 -> 3
- net col6: track 94.8 -> 283.0 mm, vias 0 -> 3
- net col7: track 94.8 -> 267.0 mm, vias 0 -> 3
- net col8: track 94.8 -> 246.3 mm, vias 0 -> 3
- net LEDGND: track 290.1 -> 441.4 mm, vias 0 -> 8
- net col9: track 115.8 -> 245.6 mm, vias 0 -> 2
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
Commit message: routing update
Parts:
- moved C7 8.74 mm to (399.7, 193.9), turned to 270 degrees
- moved C5 6.12 mm to (392.6, 193.9), turned to 270 degrees
- moved C6 4.25 mm to (397.4, 193.9), turned to 270 degrees
- moved C1 2.25 mm to (395.0, 193.9), turned to 270 degrees
Routing:
- net +5V: track 3660.3 -> 3635.1 mm, vias 8 -> 7
- net GND: track 642.4 -> 637.5 mm
- net col4: track 319.9 -> 316.7 mm
- net col7: track 267.0 -> 264.2 mm
- net col6: track 283.0 -> 280.2 mm
- net col5: track 306.1 -> 304.3 mm
Other:
- board size 324.3 x 133 mm -> 313.8 x 127.2 mm

Commit message: pcb updates
Parts:
- moved C14 276.1 mm to (427.0, 112.7)
- moved C16 276.1 mm to (431.8, 112.7)
- moved C18 276.1 mm to (436.6, 112.7)
- moved C15 276.1 mm to (429.4, 112.7)
- moved C17 276.1 mm to (434.2, 112.7)
- moved C10 7.61 mm to (134.0, 110.1)
- moved C9 7.61 mm to (131.7, 110.1)
- moved C11 7.61 mm to (136.4, 110.1)
- moved C12 7.61 mm to (138.8, 110.1)
- moved C13 7.61 mm to (141.2, 110.1)
Routing:
- net +5V: track 3635.1 -> 2545.0 mm, vias 7 -> 9
- net GND: track 637.5 -> 664.4 mm
