File: abra-PCB-v4/keyboard-5.kicad_pcb (KiCad board)
At the start: 2 copper layers, 313.8 x 127.2 mm, 294 parts, among them J2 Conn_01x04, Q1 Q_NPN_BCE, SW1 Rotary_Encoder_Switch, SW2 SW_Push, U1 ATmega32U4-AU, U2 PRTR5V0U2X, Y1 16MHz

Commit message: pcb updates
Routing:
- net +5V: track 3657.8 -> 2862.9 mm, vias 9 -> 11
- net GND: track 664.4 -> 674.7 mm
- net row0: vias 3 -> 2
