File: abra-PCB-v4/keyboard-5.sch (KiCad schematic (older format))
At the start: 294 parts, among them J2 Conn_01x04, Q1 Q_NPN_BCE, SW1 Rotary_Encoder_Switch, SW2 SW_Push, U1 ATmega32U4-AU, U2 PRTR5V0U2X, Y1 16MHz

Commit message: pcb updates
Other:
- moved on the sheet: C8, F1, J2, R4, R6, R7, R91, R92, U2, USB1
