File: abra-PCB-v4/keyboard-6.kicad_pcb (KiCad board)
At the start: 2 copper layers, 313.8 x 127.2 mm, 294 parts, among them J2 Conn_01x04, Q1 Q_NPN_BCE, SW1 Rotary_Encoder_Switch, SW2 SW_Push, U1 ATmega32U4-AU, U2 PRTR5V0U2X, Y1 16MHz

Commit message: pcb updates
Parts:
- removed the R21 at (142.1, 171.4)
- renumbered C2 to C1, C14 to C10, C15 to C11, C16 to C12, C17 to C13, C18 to C14, C1 to C15, C5 to C16, C6 to C17, C7 to C18, C3 to C2, C4 to C3, C8 to C4, C9 to C5, C10 to C6, C11 to C7, C12 to C8, C13 to C9, D_0 to D_1, D_9 to D_10, D_10 to D_11, D_11 to D_12, D_12 to D_13, D_13 to D_14, D_14 to D_15, D_15 to D_16, D_16 to D_17, D_17 to D_18, D_18 to D_19, D_1 to D_2, D_19 to D_20, D_20 to D_21, D_21 to D_22, D_22 to D_23, D_23 to D_24, D_24 to D_25, D_25 to D_26, D_26 to D_27, D_27 to D_28, D_28 to D_29, D_2 to D_3, D_29 to D_30, D_30 to D_31, D_31 to D_32, D_32 to D_33, D_33 to D_34, D_34 to D_35, D_35 to D_36, D_36 to D_37, D_37 to D_38, D_38 to D_39, D_3 to D_4, D_39 to D_40, D_40 to D_41, D_41 to D_42, D_42 to D_43, D_43 to D_44, D_4 to D_5, D_5 to D_6, D_6 to D_7, D_72 to D_71, D_71 to D_72, D_7 to D_8, D_8 to D_9, J2 to J1, K_0 to K_1, K_9 to K_10, K_10 to K_11, K_11 to K_12, K_12 to K_13, K_1 to K_2, K_2 to K_3, K_3 to K_4, K_4 to K_5, K_5 to K_6, K_6 to K_7, K_72 to K_71, K_71 to K_72, K_7 to K_8, K_8 to K_9, R11 to R1, R64 to R10, R70 to R11, R75 to R12, R81 to R13, R12 to R14, R16 to R15, R23 to R16, R28 to R17, R33 to R18, R38 to R19, R22 to R2, R44 to R20, R49 to R21, R54 to R22, R59 to R23, R65 to R24, R71 to R25, R76 to R26, R82 to R27, R86 to R28, R13 to R29, R27 to R3, R17 to R30, R24 to R31, R29 to R32, R34 to R33, R39 to R34, R45 to R35, R50 to R36, R55 to R37, R60 to R38, R66 to R39, R32 to R4, R72 to R40, R77 to R41, R83 to R42, R87 to R43, R10 to R44, R18 to R46, R93 to R47, R30 to R48, R35 to R49, R37 to R5, R40 to R50, R46 to R51, R51 to R52, R56 to R53, R61 to R54, R67 to R55, R73 to R56, R78 to R57, R88 to R58, R14 to R59, R43 to R6, R19 to R60, R25 to R61, R31 to R62, R36 to R63, R41 to R64, R47 to R65, R52 to R66, R57 to R67, R62 to R68, R68 to R69, R48 to R7, R79 to R70, R84 to R71, R89 to R72, R15 to R73, R20 to R74, R26 to R75, R42 to R76, R63 to R77, R69 to R78, R74 to R79, R53 to R8, R85 to R81, R90 to R82, R3 to R83, R2 to R84, R1 to R85, R91 to R86, R92 to R87, R6 to R88, R7 to R89, R58 to R9, R8 to R90, R4 to R91, R5 to R92, R9 to R93, U2 to U1, U1 to U2
Connections:
- K_26 pad 4: LEDGND -> Net-(K_26-Pad4)
- K_45 pad 4: Net-(K_45-Pad4) -> Net-(K_44-Pad4)
- R14 pad 2: Net-(K_41-Pad4) -> LEDGND
- R15 pad 2: Net-(K_41-Pad4) -> LEDGND
- R16 pad 2: Net-(K_41-Pad4) -> LEDGND
- R17 pad 2: Net-(K_41-Pad4) -> LEDGND
- R18 pad 2: Net-(K_41-Pad4) -> LEDGND
- R19 pad 2: Net-(K_41-Pad4) -> LEDGND
- R20 pad 2: Net-(K_41-Pad4) -> LEDGND
- R21 pad 2: Net-(K_41-Pad4) -> LEDGND
- R22 pad 2: Net-(K_41-Pad4) -> LEDGND
- R23 pad 2: Net-(K_41-Pad4) -> LEDGND
- R24 pad 2: Net-(K_41-Pad4) -> LEDGND
- R25 pad 2: Net-(K_41-Pad4) -> LEDGND
- R26 pad 1: LEDGND -> Net-(K_26-Pad4)
- R26 pad 2: Net-(K_41-Pad4) -> LEDGND
- R27 pad 2: Net-(K_41-Pad4) -> LEDGND
- R28 pad 2: Net-(K_41-Pad4) -> LEDGND
- R29 pad 2: Net-(K_57-Pad4) -> LEDGND
- R30 pad 2: Net-(K_57-Pad4) -> LEDGND
- R31 pad 2: Net-(K_57-Pad4) -> LEDGND
- R32 pad 2: Net-(K_57-Pad4) -> LEDGND
- R33 pad 2: Net-(K_57-Pad4) -> LEDGND
- R34 pad 2: Net-(K_57-Pad4) -> LEDGND
- R35 pad 2: Net-(K_57-Pad4) -> LEDGND
- R36 pad 2: Net-(K_57-Pad4) -> LEDGND
- R37 pad 2: Net-(K_57-Pad4) -> LEDGND
- R38 pad 2: Net-(K_57-Pad4) -> LEDGND
- R39 pad 2: Net-(K_57-Pad4) -> LEDGND
- R40 pad 2: Net-(K_57-Pad4) -> LEDGND
- R41 pad 2: Net-(K_57-Pad4) -> LEDGND
- R42 pad 2: Net-(K_57-Pad4) -> LEDGND
- R43 pad 2: Net-(K_57-Pad4) -> LEDGND
- R44 pad 2: Net-(K_70-Pad4) -> LEDGND
- R46 pad 2: Net-(K_70-Pad4) -> LEDGND
- R47 pad 2: Net-(K_70-Pad4) -> LEDGND
- R48 pad 2: Net-(K_70-Pad4) -> LEDGND
- R49 pad 2: Net-(K_70-Pad4) -> LEDGND
- R50 pad 2: Net-(K_70-Pad4) -> LEDGND
- R51 pad 2: Net-(K_70-Pad4) -> LEDGND
- R52 pad 2: Net-(K_70-Pad4) -> LEDGND
- R53 pad 2: Net-(K_70-Pad4) -> LEDGND
- R54 pad 2: Net-(K_70-Pad4) -> LEDGND
- R55 pad 2: Net-(K_70-Pad4) -> LEDGND
- R56 pad 2: Net-(K_70-Pad4) -> LEDGND
- R57 pad 2: Net-(K_70-Pad4) -> LEDGND
- R58 pad 2: Net-(K_70-Pad4) -> LEDGND
- R59 pad 2: Net-(K_80-Pad4) -> LEDGND
- R60 pad 2: Net-(K_80-Pad4) -> LEDGND
- R61 pad 2: Net-(K_80-Pad4) -> LEDGND
- R62 pad 2: Net-(K_80-Pad4) -> LEDGND
- R63 pad 2: Net-(K_80-Pad4) -> LEDGND
- R64 pad 2: Net-(K_80-Pad4) -> LEDGND
- R65 pad 2: Net-(K_80-Pad4) -> LEDGND
- R66 pad 2: Net-(K_80-Pad4) -> LEDGND
- R67 pad 2: Net-(K_80-Pad4) -> LEDGND
- R68 pad 2: Net-(K_80-Pad4) -> LEDGND
- R69 pad 2: Net-(K_80-Pad4) -> LEDGND
- R70 pad 2: Net-(K_80-Pad4) -> LEDGND
- R71 pad 2: Net-(K_80-Pad4) -> LEDGND
- R72 pad 2: Net-(K_80-Pad4) -> LEDGND
- R73 pad 2: Net-(R15-Pad2) -> LEDGND
- R74 pad 2: Net-(R15-Pad2) -> LEDGND
- R75 pad 2: Net-(R15-Pad2) -> LEDGND
- R76 pad 2: Net-(R15-Pad2) -> LEDGND
- R77 pad 2: Net-(R15-Pad2) -> LEDGND
- R78 pad 2: Net-(R15-Pad2) -> LEDGND
- R79 pad 2: Net-(R15-Pad2) -> LEDGND
- R80 pad 2: Net-(R15-Pad2) -> LEDGND
- R81 pad 2: Net-(R15-Pad2) -> LEDGND
- R82 pad 2: Net-(R15-Pad2) -> LEDGND
Routing:
- net +5V: track 3657.8 -> 2662.1 mm, vias 9 -> 8
- net LEDGND: track 441.4 -> 1042.3 mm
- net Net-(K_80-Pad4): track 332.7 -> 3.89 mm, vias 1 -> 0
- net Net-(R15-Pad2): track 299.2 -> 0.00 mm
- net Net-(K_45-Pad4): track 12.6 -> 0.00 mm
- net GND: track 664.4 -> 674.7 mm
- net Net-(K_70-Pad4): track 426.0 -> 416.6 mm
- net Net-(K_44-Pad4): track 3.61 -> 11.9 mm
- net row0: vias 3 -> 2
