File: abra-PCB-v4/keyboard-6.sch (KiCad schematic (older format))
At the start: 294 parts, among them J2 Conn_01x04, Q1 Q_NPN_BCE, SW1 Rotary_Encoder_Switch, SW2 SW_Push, U1 ATmega32U4-AU, U2 PRTR5V0U2X, Y1 16MHz

Commit message: pcb updates
Parts:
- removed D_0: D, Diode_SMD:D_SOD-123, symbol Device:D_Small
- removed R21: R_Small, acheron_Components:R_SMD_1206, symbol Device:R_Small
- added D_1: D, Diode_SMD:D_SOD-123, symbol Device:D_Small
- renumbered C2 to C1, C14 to C10, C15 to C11, C16 to C12, C17 to C13, C18 to C14, C1 to C15, C5 to C16, C6 to C17, C7 to C18, C3 to C2, C4 to C3, C8 to C4, C9 to C5, C10 to C6, C11 to C7, C12 to C8, C13 to C9, D_9 to D_10, D_10 to D_11, D_11 to D_12, D_12 to D_13, D_13 to D_14, D_14 to D_15, D_15 to D_16, D_16 to D_17, D_17 to D_18, D_18 to D_19, D_1 to D_2, D_19 to D_20, D_20 to D_21, D_21 to D_22, D_22 to D_23, D_23 to D_24, D_24 to D_25, D_25 to D_26, D_26 to D_27, D_27 to D_28, D_28 to D_29, D_2 to D_3, D_29 to D_30, D_30 to D_31, D_31 to D_32, D_32 to D_33, D_33 to D_34, D_34 to D_35, D_35 to D_36, D_36 to D_37, D_37 to D_38, D_38 to D_39, D_3 to D_4, D_39 to D_40, D_40 to D_41, D_41 to D_42, D_42 to D_43, D_43 to D_44, D_4 to D_5, D_5 to D_6, D_6 to D_7, D_72 to D_71, D_71 to D_72, D_7 to D_8, D_8 to D_9, J2 to J1, K_0 to K_1, K_9 to K_10, K_10 to K_11, K_11 to K_12, K_12 to K_13, K_1 to K_2, K_2 to K_3, K_3 to K_4, K_4 to K_5, K_5 to K_6, K_6 to K_7, K_72 to K_71, K_71 to K_72, K_7 to K_8, K_8 to K_9, R11 to R1, R64 to R10, R70 to R11, R75 to R12, R81 to R13, R12 to R14, R16 to R15, R23 to R16, R28 to R17, R33 to R18, R38 to R19, R22 to R2, R44 to R20, R49 to R21, R54 to R22, R59 to R23, R65 to R24, R71 to R25, R76 to R26, R82 to R27, R86 to R28, R13 to R29, R27 to R3, R17 to R30, R24 to R31, R29 to R32, R34 to R33, R39 to R34, R45 to R35, R50 to R36, R55 to R37, R60 to R38, R66 to R39, R32 to R4, R72 to R40, R77 to R41, R83 to R42, R87 to R43, R10 to R44, R18 to R46, R93 to R47, R30 to R48, R35 to R49, R37 to R5, R40 to R50, R46 to R51, R51 to R52, R56 to R53, R61 to R54, R67 to R55, R73 to R56, R78 to R57, R88 to R58, R14 to R59, R43 to R6, R19 to R60, R25 to R61, R31 to R62, R36 to R63, R41 to R64, R47 to R65, R52 to R66, R57 to R67, R62 to R68, R68 to R69, R48 to R7, R79 to R70, R84 to R71, R89 to R72, R15 to R73, R20 to R74, R26 to R75, R42 to R76, R63 to R77, R69 to R78, R74 to R79, R53 to R8, R85 to R81, R90 to R82, R3 to R83, R2 to R84, R1 to R85, R91 to R86, R92 to R87, R6 to R88, R7 to R89, R58 to R9, R8 to R90, R4 to R91, R5 to R92, R9 to R93, U2 to U1, U1 to U2
Connections:
- net LEDGND: now also R14.2, R15.2, R16.2, R17.2, R18.2, R19.2, R20.2, R21.2, R22.2, R23.2, R24.2, R25.2, R26.2, R27.2, R28.2, R29.2, R30.2, R31.2, R32.2, R33.2, R34.2, R35.2, R36.2, R37.2, R38.2, R39.2, R40.2, R41.2, R42.2, R43.2, R44.2, R46.2, R47.2, R48.2, R49.2, R50.2, R51.2, R52.2, R53.2, R54.2, R55.2, R56.2, R57.2, R58.2, R59.2, R60.2, R61.2, R62.2, R63.2, R64.2, R65.2, R66.2, R67.2, R68.2, R69.2, R70.2, R71.2, R72.2, R73.2, R74.2, R75.2, R76.2, R77.2, R78.2, R79.2, R80.2, R81.2, R82.2; no longer K_26.4 (LEDGND), R26.1
- net row0: now also D_1.1 (K)
- net at K_1.2 (ROW): now also D_1.2 (A)
- net at K_44.4 (LEDGND), R44.1: now also K_45.4 (LEDGND)
- new net: K_26.4 (LEDGND), R26.1
- new net: K_41.4 (LEDGND), R41.1
- new net: K_57.4 (LEDGND), R57.1
- new net: K_70.4 (LEDGND), R70.1
- new net: K_80.4 (LEDGND), R80.1
Other:
- moved on the sheet: C1, C10, C11, C12, C13, C14, C15, C16, C17, C18, C2, C3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
