File: abra-PCB-v4/keyboard-8.kicad_pcb (KiCad board)
At the start: 2 copper layers, 313.8 x 124.8 mm, 214 parts, among them SW1 Rotary_Encoder_Switch, SW2 SW_Push, U1 PRTR5V0U2X, U2 ATmega32U4-AU, Y1 16MHz

Commit message: gerber export
Parts:
- moved C15 1.70 mm to (407.4, 172.7)
Routing:
- net col3: track 305.1 -> 294.2 mm, vias 2 -> 0
- net col1: track 349.6 -> 344.4 mm
- net col2: track 346.6 -> 342.0 mm
- net RGBIN: track 365.5 -> 361.6 mm
- net +5V: track 1701.1 -> 1703.8 mm
- net col0: track 401.9 -> 400.0 mm
- net GND: track 761.8 -> 763.5 mm
- net col4: track 316.7 -> 317.9 mm
