File: abra-PCB-v4/keyboard-9.kicad_pcb (KiCad board)
At the start: 2 copper layers, 313.8 x 124.8 mm, 214 parts, among them SW1 Rotary_Encoder_Switch, SW2 SW_Push, U1 PRTR5V0U2X, U2 ATmega32U4-AU, Y1 16MHz

Commit message: gerber export
Parts:
- added D11: SK6812, EC15-LED_SMD:LED_SK6812_EC15_1.5x1.5mm, F.Cu at (133.9, 140.4)
- D1, D10, D2, D3, D4, D5, D6, D7, D8, D9: footprint LED_SMD:LED_SK6812_EC15_1.5x1.5mm -> EC15-LED_SMD:LED_SK6812_EC15_1.5x1.5mm
Routing:
- net +5V: track 1708.2 -> 1695.7 mm
