File: abra-PCB-v4/keyboard-9.sch (KiCad schematic (older format))
At the start: 214 parts, among them SW1 Rotary_Encoder_Switch, SW2 SW_Push, U1 PRTR5V0U2X, U2 ATmega32U4-AU, Y1 16MHz

Commit message: gerber export
Parts:
- removed D1, D10, D2, D3, D4, D5, D6, D7, D8, D9: SK6805, LED_SMD:LED_SK6812_EC15_1.5x1.5mm, symbol LED:SK6805
- added D? (x10): SK6805-EC15, LED_SMD:LED_SK6805_PLCC4_2.4x2.7mm_P1.3mm, symbol EC15-LED:SK6805-EC15
Other:
- moved on the sheet: R10
