File: abra-PCB-v4/keyboard-10.kicad_pcb (KiCad board)
At the start: 2 copper layers, 313.8 x 124.8 mm, 214 parts, among them SW2 Rotary_Encoder_Switch, U1 PRTR5V0U2X, U2 ATmega32U4-AU, Y1 16MHz

Commit message: backspace fix led spacing update
Parts:
- K_27: footprint MX_Only:MXOnly-1U-NoLED -> MX_Only:MXOnly-2U-NoLED
- moved C6 11.0 mm to (131.2, 128.0)
- moved D1 11.0 mm to (128.6, 127.7)
- moved C11 10.8 mm to (437.1, 128.0)
- moved D6 10.7 mm to (439.2, 127.7)
- moved R8 8.87 mm to (129.0, 121.5)
- moved C12 7.37 mm to (437.1, 141.0)
- moved C7 6.48 mm to (131.0, 142.0)
- moved D2 6.48 mm to (128.7, 141.7)
- moved D7 6.10 mm to (439.2, 141.8)
- moved C8 3.94 mm to (131.1, 154.1)
- moved D3 3.94 mm to (128.8, 153.9)
- moved C13 3.69 mm to (437.1, 154.3)
- moved D8 3.62 mm to (439.2, 154.0)
- moved D10 2.99 mm to (439.1, 179.6)
- moved C10 2.80 mm to (131.3, 180.0)
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Routing:
- net +5V: track 716.4 -> 689.1 mm
- net GND: track 272.8 -> 255.3 mm, vias 15 -> 18
- net Net-(D5-Pad3): track 450.9 -> 441.1 mm, vias 2 -> 3
- net RGBIN: track 339.9 -> 331.3 mm
- net col13: track 221.0 -> 213.2 mm
- net col11: track 213.2 -> 219.2 mm
- net ENS: track 119.8 -> 114.6 mm
- net Net-(D6-Pad3): track 9.02 -> 13.9 mm
- net Net-(D8-Pad3): track 8.81 -> 13.6 mm
- net col10: track 232.0 -> 236.6 mm
- net Net-(D1-Pad3): track 8.96 -> 13.4 mm
- net row5: track 353.8 -> 349.6 mm
- net Net-(D3-Pad3): track 8.78 -> 12.7 mm
- net VCC: track 65.7 -> 62.7 mm
- net Net-(D7-Pad3): track 9.18 -> 12.0 mm
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