File: abra-PCB-v4/keyboard-10.sch (KiCad schematic (older format))
At the start: 214 parts, among them SW2 Rotary_Encoder_Switch, U1 PRTR5V0U2X, U2 ATmega32U4-AU, Y1 16MHz

Commit message: backspace fix led spacing update
Parts:
- K_27: footprint MX_Only:MXOnly-1U-NoLED -> MX_Only:MXOnly-2U-NoLED
- S1: renamed from S?; footprint SW_EVP-BB2A9B000 -> EVP-BB2A9B000:SW_EVP-BB2A9B000
Changed lines of the file:
@@
 F 0 "K_27" H 20150 2583 60  0000 C CNN
 F 1 "KEYSW" H 20150 2250 60  0001 C CNN
-F 2 "MX_Only:MXOnly-1U-NoLED" H 20150 2350 60  0001 C CNN
+F 2 "MX_Only:MXOnly-2U-NoLED" H 20150 2350 60  0001 C CNN
 F 3 "" H 20150 2350 60  0000 C CNN
 	1    20150 2350
@@
 	19150 12200 19450 12200
 $Comp
-L EVP-BB2A9B000:EVP-BB2A9B000 S?
+L EVP-BB2A9B000:EVP-BB2A9B000 S1
 U 1 1 5F6F7B9A
 P 1700 10350
-F 0 "S?" H 1700 10631 50  0000 C CNN
+F 0 "S1" H 1700 10631 50  0000 C CNN
 F 1 "EVP-BB2A9B000" H 1700 10540 50  0000 C CNN
-F 2 "SW_EVP-BB2A9B000" H 1700 10350 50  0001 L BNN
+F 2 "EVP-BB2A9B000:SW_EVP-BB2A9B000" H 1700 10350 50  0001 L BNN
 F 3 "EVP-BB2A9B000" H 1700 10350 50  0001 L BNN
 F 4 "Tactile Switch SPST-NO Top Actuated Surface Mount" H 1700 10350 50  0001 L BNN "Field4"
